File: FumeDisperser.sch (EAGLE design)
At the start: 19 parts, among them IC1 MC34063AD

Commit message: Add PWM controller circuit
Parts:
- added C4, C6, C8: 0.1, resistor:C-EUC1206
- added C5: 10uF, rcl:CPOL-EUD/7343-31R
- added C7: 220uF, rcl:CPOL-EUD/7343-31R
- added D2, D3: (no value), adafruit:DIODESOD-123
- added IC2: NE555D, linear:NE555D
- added PAD7: Fan_PWM, wirepad:SMD5
- added R10, R8, R9: 1k, resistor:R-EU_M1206
- added R11: 47k, resistor:R-EU_M1206
- added R12, R13: 0, resistor:R-EU_M1206
- added R6: 30k, resistor:R-EU_M1206
- added R7: 150k, resistor:R-EU_M1206
- added T1: bc817, transistor:BC817-16-NPN-SOT23-BEC
- R1: value 2.2k -> 3.9k
- R2: value 12k -> 33k
Connections:
- new net N$27: R13.1, R5.S
- new net N$29: C7.+, IC2.R, R6.2, R7.1
- new net N$30: D3.C, R8.1
- new net N$31: D2.A, R9.1
- new net N$32: R5.E, R9.2
- new net N$33: R5.A, R8.2
- new net N$34: IC2.Q, R13.2
- new net N$35: IC2.DIS, R10.1
- new net N$36: R10.2, R11.1, T1.B
- new net N$37: PAD7.P, T1.C
- new net N$42: R12.2, T1.E
- new net VCC: C1.+, C4.1, C5.+, D1.C, IC2.V+, PAD6.P, R11.2, R2.2, R7.2
- net GND: now also C4.2, C5.-, C6.2, C7.-, C8.2, IC2.GND, R12.1, R6.1
- net N$11: now also C8.1, D2.C, D3.A, IC2.THR, IC2.TR; no longer R2.2, R5.A, R5.S
- net N$2: now also C6.1, IC2.CV; no longer C1.+, D1.C, PAD6.P, R5.E
Other:
- moved on the sheet: R5
